File: file60144165.sch (KiCad schematic (older format))
At the start: 30 parts, among them U2 IS31FL3737, U4 IS31FL3737

Commit message: test
Parts:
- removed JP1, JP3: Right, Keyboard 2:SolderJumper-2_P1.3mm_Open_TrianglePad1.0x1.5mm, symbol Jumper:SolderJumper_2_Open
- removed JP2, JP4: Left, Keyboard 2:SolderJumper-2_P1.3mm_Open_TrianglePad1.0x1.5mm, symbol Jumper:SolderJumper_2_Open
- removed R3, R5: 100k, Resistor_SMD:R_0603_1608Metric, symbol Device:R
- added R7: 1k, Resistor_SMD:R_0603_1608Metric, symbol Device:R
- R6: value 100k -> 1k
Connections:
- net GND: now also U4.36 (ADDR); no longer R6.1
- net I2C+: now also R6.2
- net I2C-: now also R7.1
- net RGB_SYNC: now reaches U2.33 (SYNC)
- net RGB_SYNC: now also U4.33 (SYNC)
- net PWR: now reaches U2.36 (ADDR)
- net PWR: now also C1.2, C15.2, C17.1, C18.2, C19.2, C2.2, C20.2, C21.2, C22.2, C3.2, C4.2, C5.1, C6.2, C7.2, U2.19 (PVCC), U2.26 (PVCC), U2.31 (VCC), U4.19 (PVCC), U4.26 (PVCC), U4.31 (VCC)
- net RGB_ENABLE renamed SDB
- net SDB: no longer R6.2
- net RGB_INT renamed INTB
- net INTB: no longer U2.37 (~INTB)
- net RSET: no longer names the net of R4.2, U2.30 (RSET)
- net RSET: no longer R14.2, U4.30 (RSET)
- removed net VCC: C1.2, C15.2, C16.2, C17.1, C18.2, C19.2, C2.2, C20.2, C21.2, C22.2, C3.2, C4.2, C5.1, C6.2, C7.2, C8.2, U2.19 (PVCC), U2.26 (PVCC), U2.31 (VCC), U2.32 (VIO), U4.19 (PVCC), U4.26 (PVCC), U4.31 (VCC), U4.32 (VIO)
- new net: R14.2, U4.30 (RSET)
- new net V_IO: C16.2, C8.2, R6.1, R7.2, U2.32 (VIO), U4.32 (VIO)
- no-connect marks 2 -> 1
Other:
- note added: "Sync Master"
- note added: "Sync Slave"
- moved on the sheet: R14, R15, R16, R17
