File: file60149CD6.sch (KiCad schematic (older format))
At the start: 96 parts

Commit message: Added wireless circuit
nRF82840 wirelss module
TP4056 Charging/loadshare
Other:
- moved on the sheet: RGB_1, RGB_10, RGB_11, RGB_12, RGB_13, RGB_14, RGB_15, RGB_16, RGB_17, RGB_18, RGB_19, RGB_2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

Commit message: test
Parts:
- added RGB_5B1: RGB, Keyboard Library:APTF1616SEEZGQBDC, symbol Device:LED_ARGB
Connections:
- wire segments 1064 -> 1073
Other:
- moved on the sheet: RGB_1, RGB_10, RGB_11, RGB_12, RGB_13, RGB_14, RGB_15, RGB_16, RGB_17, RGB_18, RGB_19, RGB_2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
