File: yurei.kicad_pcb (KiCad board)
At the start: 2 copper layers, 345 x 122 mm, 183 parts, among them SW1 SW_SPST, SW10 SW_SPST, SW11 SW_SPST, SW12 SW_SPST, SW13 SW_SPST, SW14 SW_SPST, SW15 SW_SPST, SW16 SW_SPST, SW17 SW_SPST, SW18 SW_SPST, SW19 SW_SPST, SW2 SW_SPST, SW20 SW_SPST, SW21 SW_SPST, SW22 SW_SPST, SW23 SW_SPST, SW24 SW_SPST, SW25 SW_SPST, SW26 SW_SPST, SW27 SW_SPST, SW28 SW_SPST, SW29 SW_SPST, SW3 SW_SPST, SW30 SW_SPST, SW31 SW_SPST, SW32 SW_SPST, SW33 SW_SPST, SW34 SW_SPST, SW35 SW_SPST, SW36 SW_SPST, SW37 SW_SPST, SW38 SW_SPST, SW39 SW_SPST, SW4 SW_SPST, SW40 SW_SPST, SW41 SW_SPST, SW42 SW_SPST, SW43 SW_SPST, SW44 SW_SPST, SW45 SW_SPST, SW46 SW_SPST, SW47 SW_SPST, SW48 SW_SPST, SW49 SW_SPST, SW5 SW_SPST, SW50 SW_SPST, SW51 SW_SPST, SW52 SW_SPST, SW53 SW_SPST, SW54 SW_SPST, SW55 SW_SPST, SW56 SW_SPST, SW57 SW_SPST, SW58 SW_SPST, SW59 SW_SPST, SW6 SW_SPST, SW60 SW_SPST, SW61 SW_SPST, SW62 SW_SPST, SW63 SW_SPST, SW64 SW_SPST, SW65 SW_SPST, SW66 SW_SPST, SW67 SW_SPST, SW68 SW_SPST, SW69 SW_SPST, SW7 SW_SPST, SW70 SW_SPST, SW71 SW_SPST, SW72 SW_SPST, SW73 SW_SPST, SW74 SW_SPST, SW75 SW_SPST, SW76 SW_SPST, SW77 SW_SPST, SW78 SW_SPST, SW79 SW_SPST, SW8 SW_SPST, SW80 SW_SPST, SW81 SW_SPST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

Commit message: First edit
Parts:
- removed U1: Teensy2.0_(C), yurei:Teensy2.0
- removed kicad1, kicad2: KiCad-Logo2_5mm_SilkScreen, yurei:KiCad-Logo2_5mm_SilkScreen
- removed oshw1, oshw2: OSHW-Logo_7.5x8mm_SilkScreen, yurei:OSHW-Logo_7.5x8mm_SilkScreen
- added C1: 0u1, Capacitor_SMD:C_0603_1608Metric, F.Cu at (338.7, 143.7)
- added C15: 0u1, Capacitor_SMD:C_0603_1608Metric, F.Cu at (127.0, 94.2)
- added C16: 0u47, Capacitor_SMD:C_0603_1608Metric, F.Cu at (119.0, 91.7)
- added C17: 22uF 10V, Capacitor_Tantalum_SMD:CP_EIA-3216-18_Kemet-A, F.Cu at (112.6, 99.3)
- added C18: 0u1, Capacitor_SMD:C_0603_1608Metric, F.Cu at (125.4, 99.2)
- added C19: 0u1, Capacitor_SMD:C_0603_1608Metric, F.Cu at (121.4, 99.2)
- added C2: 0u47, Capacitor_SMD:C_0603_1608Metric, F.Cu at (338.7, 146.2)
- added C20: 0u47, Capacitor_SMD:C_0603_1608Metric, F.Cu at (121.4, 96.7)
- added C21: 0u47, Capacitor_SMD:C_0603_1608Metric, F.Cu at (125.4, 96.7)
- added C22: 0u47, Capacitor_SMD:C_0603_1608Metric, F.Cu at (127.0, 91.7)
- added C3: 0u1, Capacitor_SMD:C_0603_1608Metric, F.Cu at (337.1, 151.0)
- added C4: 0u47, Capacitor_SMD:C_0603_1608Metric, F.Cu at (342.7, 143.7)
- added C5: 22uF 10V, Capacitor_Tantalum_SMD:CP_EIA-3216-18_Kemet-A, F.Cu at (332.2, 151.3)
- added C6: 0u1, Capacitor_SMD:C_0603_1608Metric, F.Cu at (342.7, 146.2)
- added C7: 0u47, Capacitor_SMD:C_0603_1608Metric, F.Cu at (346.7, 143.7)
- added C8: 0u47, Capacitor_SMD:C_0603_1608Metric, F.Cu at (341.1, 148.8)
- added R14: 20k, Resistor_SMD:R_0603_1608Metric, F.Cu at (123.0, 94.2)
- added R15: 100k, Resistor_SMD:R_0603_1608Metric, F.Cu at (123.0, 91.7)
- added R16: 100k, Resistor_SMD:R_0603_1608Metric, F.Cu at (117.4, 99.0)
- added R17: 100k, Resistor_SMD:R_0603_1608Metric, F.Cu at (119.0, 94.2)
- added R3: 100k, Resistor_SMD:R_0603_1608Metric, F.Cu at (346.7, 146.2)
- added R4: 20k, Resistor_SMD:R_0603_1608Metric, F.Cu at (341.1, 151.3)
- added R5: 100k, Resistor_SMD:R_0603_1608Metric, F.Cu at (345.1, 148.8)
- added R6: 100k, Resistor_SMD:R_0603_1608Metric, F.Cu at (345.1, 151.3)
- added RGB_1: RGB, Keyboard Library:APTF1616SEEZGQBDC, F.Cu at (45.4, 87.0)
- added RGB_10: RGB, Keyboard Library:APTF1616SEEZGQBDC, F.Cu at (78.9, 152.9)
- added RGB_11: RGB, Keyboard Library:APTF1616SEEZGQBDC, F.Cu at (88.4, 172.2)
- added RGB_12: RGB, Keyboard Library:APTF1616SEEZGQBDC, F.Cu at (71.6, 191.2)
- added RGB_13: RGB, Keyboard Library:APTF1616SEEZGQBDC, F.Cu at (83.5, 87.0)
- added RGB_14: RGB, Keyboard Library:APTF1616SEEZGQBDC, F.Cu at (83.6, 114.8)
- added RGB_15: RGB, Keyboard Library:APTF1616SEEZGQBDC, F.Cu at (93.3, 133.9)
- added RGB_16: RGB, Keyboard Library:APTF1616SEEZGQBDC, F.Cu at (97.8, 153.1)
- added RGB_17: RGB, Keyboard Library:APTF1616SEEZGQBDC, F.Cu at (107.3, 172.2)
- added RGB_18: RGB, Keyboard Library:APTF1616SEEZGQBDC, F.Cu at (95.7, 191.2)
- added RGB_19: RGB, Keyboard Library:APTF1616SEEZGQBDC, F.Cu at (102.5, 86.8)
- added RGB_2: RGB, Keyboard Library:APTF1616SEEZGQBDC, F.Cu at (45.6, 115.0)
- added RGB_20: RGB, Keyboard Library:APTF1616SEEZGQBDC, F.Cu at (102.4, 114.6)
- added RGB_21: RGB, Keyboard Library:APTF1616SEEZGQBDC, F.Cu at (111.8, 133.9)
- added RGB_22: RGB, Keyboard Library:APTF1616SEEZGQBDC, F.Cu at (116.5, 153.4)
- added RGB_23: RGB, Keyboard Library:APTF1616SEEZGQBDC, F.Cu at (126.3, 172.1)
- added RGB_24: RGB, Keyboard Library:APTF1616SEEZGQBDC, F.Cu at (179.9, 231.7)
- added RGB_25: RGB, Keyboard Library:APTF1616SEEZGQBDC, F.Cu at (121.6, 86.9)
- added RGB_26: RGB, Keyboard Library:APTF1616SEEZGQBDC, F.Cu at (121.6, 114.8)
- added RGB_27: RGB, Keyboard Library:APTF1616SEEZGQBDC, F.Cu at (131.2, 134.0)
- added RGB_28: RGB, Keyboard Library:APTF1616SEEZGQBDC, F.Cu at (135.7, 153.0)
- added RGB_29: RGB, Keyboard Library:APTF1616SEEZGQBDC, F.Cu at (145.4, 172.2)
- added RGB_3: RGB, Keyboard Library:APTF1616SEEZGQBDC, F.Cu at (49.3, 134.0)
- added RGB_30: RGB, Keyboard Library:APTF1616SEEZGQBDC, F.Cu at (141.7, 238.0)
- added RGB_31: RGB, Keyboard Library:APTF1616SEEZGQBDC, F.Cu at (140.5, 87.5)
- added RGB_32: RGB, Keyboard Library:APTF1616SEEZGQBDC, F.Cu at (140.6, 114.9)
- added RGB_33: RGB, Keyboard Library:APTF1616SEEZGQBDC, F.Cu at (150.2, 134.0)
- added RGB_34: RGB, Keyboard Library:APTF1616SEEZGQBDC, F.Cu at (154.9, 153.1)
- added RGB_35: RGB, Keyboard Library:APTF1616SEEZGQBDC, F.Cu at (164.3, 172.0)
- added RGB_36: RGB, Keyboard Library:APTF1616SEEZGQBDC, F.Cu at (166.9, 190.9)
- added RGB_37: RGB, Keyboard Library:APTF1616SEEZGQBDC, F.Cu at (169.2, 86.9)
- added RGB_38: RGB, Keyboard Library:APTF1616SEEZGQBDC, F.Cu at (159.6, 115.0)
- added RGB_39: RGB, Keyboard Library:APTF1616SEEZGQBDC, F.Cu at (169.3, 133.8)
- added RGB_4: RGB, Keyboard Library:APTF1616SEEZGQBDC, F.Cu at (52.7, 153.3)
- added RGB_40: RGB, Keyboard Library:APTF1616SEEZGQBDC, F.Cu at (174.2, 153.0)
- added RGB_41: RGB, Keyboard Library:APTF1616SEEZGQBDC, F.Cu at (183.4, 171.7)
- added RGB_42: RGB, Keyboard Library:APTF1616SEEZGQBDC, F.Cu at (170.7, 241.9)
- added RGB_43: RGB, Keyboard Library:APTF1616SEEZGQBDC, F.Cu at (188.5, 86.9)
- added RGB_44: RGB, Keyboard Library:APTF1616SEEZGQBDC, F.Cu at (178.5, 114.8)
- added RGB_45: RGB, Keyboard Library:APTF1616SEEZGQBDC, F.Cu at (188.4, 133.9)
- added RGB_46: RGB, Keyboard Library:APTF1616SEEZGQBDC, F.Cu at (193.4, 153.1)
- added RGB_47: RGB, Keyboard Library:APTF1616SEEZGQBDC, F.Cu at (202.5, 172.3)
- added RGB_48: RGB, Keyboard Library:APTF1616SEEZGQBDC, F.Cu at (184.0, 237.0)
- added RGB_49: RGB, Keyboard Library:APTF1616SEEZGQBDC, F.Cu at (207.4, 86.9)
- added RGB_5: RGB, Keyboard Library:APTF1616SEEZGQBDC, F.Cu at (57.7, 171.7)
- added RGB_50: RGB, Keyboard Library:APTF1616SEEZGQBDC, F.Cu at (198.1, 115.0)
- added RGB_51: RGB, Keyboard Library:APTF1616SEEZGQBDC, F.Cu at (207.7, 134.0)
- added RGB_52: RGB, Keyboard Library:APTF1616SEEZGQBDC, F.Cu at (212.1, 153.1)
- added RGB_53: RGB, Keyboard Library:APTF1616SEEZGQBDC, F.Cu at (222.1, 171.9)
- added RGB_54: RGB, Keyboard Library:APTF1616SEEZGQBDC, F.Cu at (192.4, 239.1)
- added RGB_55: RGB, Keyboard Library:APTF1616SEEZGQBDC, F.Cu at (226.2, 86.9)
- added RGB_56: RGB, Keyboard Library:APTF1616SEEZGQBDC, F.Cu at (216.7, 115.0)
- added RGB_57: RGB, Keyboard Library:APTF1616SEEZGQBDC, F.Cu at (226.3, 134.0)
- added RGB_58: RGB, Keyboard Library:APTF1616SEEZGQBDC, F.Cu at (230.8, 153.1)
- added RGB_59: RGB, Keyboard Library:APTF1616SEEZGQBDC, F.Cu at (241.0, 172.1)
- added RGB_6: RGB, Keyboard Library:APTF1616SEEZGQBDC, F.Cu at (47.6, 191.1)
- added RGB_60: RGB, Keyboard Library:APTF1616SEEZGQBDC, F.Cu at (238.3, 191.1)
- added RGB_61: RGB, Keyboard Library:APTF1616SEEZGQBDC, F.Cu at (254.9, 87.0)
- added RGB_62: RGB, Keyboard Library:APTF1616SEEZGQBDC, F.Cu at (235.9, 114.8)
- added RGB_63: RGB, Keyboard Library:APTF1616SEEZGQBDC, F.Cu at (245.3, 134.0)
- added RGB_64: RGB, Keyboard Library:APTF1616SEEZGQBDC, F.Cu at (249.9, 153.2)
- added RGB_65: RGB, Keyboard Library:APTF1616SEEZGQBDC, F.Cu at (259.7, 172.0)
- added RGB_66: RGB, Keyboard Library:APTF1616SEEZGQBDC, F.Cu at (261.8, 190.8)
- added RGB_67: RGB, Keyboard Library:APTF1616SEEZGQBDC, F.Cu at (274.4, 86.8)
- added RGB_68: RGB, Keyboard Library:APTF1616SEEZGQBDC, F.Cu at (255.3, 114.4)
- added RGB_69: RGB, Keyboard Library:APTF1616SEEZGQBDC, F.Cu at (264.1, 134.0)
- added RGB_7: RGB, Keyboard Library:APTF1616SEEZGQBDC, F.Cu at (157.4, 239.4)
- added RGB_70: RGB, Keyboard Library:APTF1616SEEZGQBDC, F.Cu at (269.3, 153.1)
- added RGB_71: RGB, Keyboard Library:APTF1616SEEZGQBDC, F.Cu at (161.7, 229.1)
- added RGB_72: RGB, Keyboard Library:APTF1616SEEZGQBDC, F.Cu at (164.6, 234.2)
- added RGB_73: RGB, Keyboard Library:APTF1616SEEZGQBDC, F.Cu at (293.1, 86.9)
- added RGB_74: RGB, Keyboard Library:APTF1616SEEZGQBDC, F.Cu at (273.9, 114.9)
- added RGB_75: RGB, Keyboard Library:APTF1616SEEZGQBDC, F.Cu at (283.5, 133.8)
- added RGB_76: RGB, Keyboard Library:APTF1616SEEZGQBDC, F.Cu at (300.1, 153.1)
- added RGB_77: RGB, Keyboard Library:APTF1616SEEZGQBDC, F.Cu at (295.5, 172.3)
- added RGB_78: RGB, Keyboard Library:APTF1616SEEZGQBDC, F.Cu at (286.0, 191.2)
- added RGB_79: RGB, Keyboard Library:APTF1616SEEZGQBDC, F.Cu at (312.0, 86.8)
- added RGB_8: RGB, Keyboard Library:APTF1616SEEZGQBDC, F.Cu at (64.4, 114.9)
- added RGB_80: RGB, Keyboard Library:APTF1616SEEZGQBDC, F.Cu at (302.6, 115.0)
- added RGB_81: RGB, Keyboard Library:APTF1616SEEZGQBDC, F.Cu at (307.3, 134.1)
- added RGB_82: RGB, Keyboard Library:APTF1616SEEZGQBDC, F.Cu at (167.5, 227.8)
- added RGB_83: RGB, Keyboard Library:APTF1616SEEZGQBDC, F.Cu at (309.6, 191.2)
- added RGB_84: RGB, Keyboard Library:APTF1616SEEZGQBDC, F.Cu at (336.2, 87.0)
- added RGB_85: RGB, Keyboard Library:APTF1616SEEZGQBDC, F.Cu at (336.3, 115.1)
- added RGB_86: RGB, Keyboard Library:APTF1616SEEZGQBDC, F.Cu at (336.4, 134.0)
- added RGB_87: RGB, Keyboard Library:APTF1616SEEZGQBDC, F.Cu at (336.2, 191.1)
- added RGB_88: RGB, Keyboard Library:APTF1616SEEZGQBDC, F.Cu at (355.2, 87.0)
- added RGB_89: RGB, Keyboard Library:APTF1616SEEZGQBDC, F.Cu at (355.1, 115.0)
- added RGB_9: RGB, Keyboard Library:APTF1616SEEZGQBDC, F.Cu at (73.8, 133.9)
- added RGB_90: RGB, Keyboard Library:APTF1616SEEZGQBDC, F.Cu at (355.4, 134.2)
- added RGB_91: RGB, Keyboard Library:APTF1616SEEZGQBDC, F.Cu at (355.1, 171.4)
- added RGB_92: RGB, Keyboard Library:APTF1616SEEZGQBDC, F.Cu at (355.2, 191.2)
- added RGB_93: RGB, Keyboard Library:APTF1616SEEZGQBDC, F.Cu at (374.3, 87.1)
- added RGB_94: RGB, Keyboard Library:APTF1616SEEZGQBDC, F.Cu at (374.1, 115.1)
- added RGB_95: RGB, Keyboard Library:APTF1616SEEZGQBDC, F.Cu at (373.7, 133.9)
- added RGB_96: RGB, Keyboard Library:APTF1616SEEZGQBDC, F.Cu at (374.3, 191.2)
- added U2: IS31FL3737, Package_DFN_QFN:QFN-40-1EP_5x5mm_P0.4mm_EP3.8x3.8mm_ThermalVias, F.Cu at (333.0, 146.1)
- added U3: Core51822B, Keyboard Library:Core51822(B), B.Cu at (375.4, 147.5)
- added U4: IS31FL3737, Package_DFN_QFN:QFN-40-1EP_5x5mm_P0.4mm_EP3.8x3.8mm_ThermalVias, F.Cu at (113.4, 94.1)
- D1, D10, D11, D12, D13, D14, D15, D16, D17, D18, D19, D2, D20, D21, D22, D23, D24, D25, D26, D27, D28, D29, D3, D30, D31, D32, D33, D34, D35, D36, D37, D38, D39, D4, D40, D41, D42, D43, D44, D45, D46, D47, D48, D49, D5, D50, D51, D52, D53, D54, D55, D56, D57, D58, D59, D6, D60, D61, D62, D63, D64, D65, D66, D67, D68, D69, D7, D70, D71, D72, D73, D74, D75, D76, D77, D78, D79, D8, D80, D81, D82, D83, D84, D85, D86, D87, D9: value 1N4148 -> 1N4148W; footprint yurei:D_DO-35_SOD27_P7.62mm_Horizontal -> Diode_SMD:D_SOD-123
- SW1, SW10, SW11, SW12, SW13, SW14, SW15, SW16, SW17, SW18, SW19, SW2, SW20, SW21, SW22, SW23, SW24, SW25, SW26, SW27, SW28, SW29, SW3, SW31, SW32, SW33, SW35, SW36, SW37, SW38, SW39, SW4, SW40, SW41, SW42, SW43, SW44, SW45, SW46, SW48, SW49, SW5, SW50, SW52, SW53, SW54, SW55, SW56, SW57, SW58, SW59, SW6, SW60, SW61, SW62, SW65, SW66, SW67, SW68, SW69, SW7, SW70, SW71, SW72, SW73, SW74, SW76, SW8, SW85, SW86, SW87, SW9: footprint yurei:SW_Cherry_MX_1.00u_PCB -> keyswitches:Kailh_socket_MX_RGB
- SW30: footprint yurei:SW_Cherry_MX_2.00u_PCB -> keyswitches:Kailh_socket_MX_RGB
- SW34, SW47: footprint yurei:SW_Cherry_MX_1.50u_PCB -> keyswitches:Kailh_socket_MX_RGB
- SW51: footprint yurei:SW_Cherry_MX_1.75u_PCB -> keyswitches:Kailh_socket_MX_RGB
- SW63, SW64: footprint yurei:SW_Cherry_MX_2.25u_PCB -> keyswitches:Kailh_socket_MX_RGB
- SW75: footprint yurei:SW_Cherry_MX_2.75u_PCB -> keyswitches:Kailh_socket_MX_RGB
- SW77, SW78, SW79, SW81, SW82, SW83, SW84: footprint yurei:SW_Cherry_MX_1.25u_PCB -> keyswitches:Kailh_socket_MX_RGB
- SW80: footprint yurei:SW_Cherry_MX_6.25u_PCB -> keyswitches:Kailh_socket_MX_RGB
- moved SW42 5.68 mm to (207.3, 129.0)
- moved SW45 5.68 mm to (264.5, 129.0)
- moved SW46 5.68 mm to (283.5, 129.0)
- moved SW47 5.68 mm to (307.3, 129.0)
- moved SW48 5.68 mm to (336.1, 129.0)
- moved SW49 5.68 mm to (355.2, 129.0)
- moved SW50 5.68 mm to (374.2, 129.0)
- moved SW71 5.68 mm to (202.6, 167.1)
- moved SW74 5.68 mm to (259.7, 167.1)
- moved SW75 5.68 mm to (295.4, 167.1)
- moved SW76 5.68 mm to (355.2, 167.1)
- moved SW34 5.68 mm to (50.2, 129.0)
- moved SW36 5.68 mm to (93.0, 129.0)
- moved SW65 5.68 mm to (88.3, 167.1)
- moved SW64 5.68 mm to (57.4, 167.1)
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Routing:
- net (no net): track 0.00 -> 2374.6 mm
- net Col16: track 362.5 -> 28.0 mm
- net Col15: track 341.2 -> 104.2 mm
- net Row5: track 419.3 -> 200.7 mm
- net Col14: track 318.3 -> 104.2 mm
- net Net-(D80-Pad2): track 14.0 -> 218.6 mm
- net Col12: track 320.7 -> 137.5 mm
- net Col6: track 155.5 -> 325.3 mm, vias 0 -> 1
- net Col7: track 169.9 -> 0.00 mm, vias 1 -> 0
- net Col1: track 165.9 -> 0.00 mm
- net Row4: track 378.7 -> 279.5 mm
- net Net-(D67-Pad2): track 14.0 -> 99.2 mm
- net Col0: track 185.0 -> 113.4 mm
- net Col2: track 154.2 -> 89.2 mm
- net Row0: track 312.6 -> 274.5 mm
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
Commit message: Added wireless circuit
nRF82840 wirelss module
TP4056 Charging/loadshare
Parts:
- removed L1, L2: LED, yurei:LED_D3.0mm
- removed R1, R2: 10k, yurei:R_Axial_DIN0207_L6.3mm_D2.5mm_P7.62mm_Horizontal
- removed U3: Core51822B, Keyboard Library:Core51822(B)
- added D88: MBRS130LT3G, SamacSys_Parts:DIOM5436X247N, F.Cu at (140.6, 93.8)
- added IC1: DMP1045U-7, SamacSys_Parts:SOT96P240X120-3N, F.Cu at (147.1, 93.4)
- added P1: USB_C_Plug_USB2.0, Keyboard Library:HRO-TYPE-C-31-M-12-Assembly, B.Cu at (154.7, 73.0)
- added R7: 100k, Resistor_SMD:R_0805_2012Metric_Pad1.15x1.40mm_HandSolder, F.Cu at (136.9, 98.1)
- added RF1: HolyIOT-18010-nRF52840, Keyboard Library:HolyIOT-18010-nRF52840, F.Cu at (240.7, 82.9)
- added U5: TP4056_1A_Charge, Keyboard Library:T4056 1A Charge, B.Cu at (142.4, 93.1)
- moved C16 87.9 mm to (126.0, 179.3)
- moved C18 87.9 mm to (132.4, 186.9)
- moved C19 87.9 mm to (128.4, 186.9)
- moved C20 87.9 mm to (128.4, 184.4)
- moved C21 87.9 mm to (132.4, 184.4)
- moved C22 87.9 mm to (134.0, 179.3)
- moved R15 87.9 mm to (130.0, 179.3)
- moved C15 87.9 mm to (134.0, 181.8)
- moved C17 87.9 mm to (119.6, 186.9)
- moved R14 87.9 mm to (130.0, 181.8)
- moved R16 87.9 mm to (124.4, 186.6)
- moved R17 87.9 mm to (126.0, 181.8)
- moved U4 87.9 mm to (120.4, 181.7)
- moved RGB_54 37.4 mm to (171.7, 208.0)
- moved RGB_7 34.5 mm to (151.1, 205.4)
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Routing:
- net (no net): track 2374.6 -> 0.00 mm
- net Col6: track 325.3 -> 0.00 mm, vias 1 -> 0
- net Row1: track 309.6 -> 0.00 mm
- net Row2: track 304.8 -> 0.00 mm
- net Row3: track 303.3 -> 0.00 mm
- net Col13: track 283.2 -> 0.00 mm, vias 1 -> 0
- net Row4: track 279.5 -> 0.00 mm
- net Row0: track 274.5 -> 0.00 mm
- net Col11: track 268.5 -> 0.00 mm, vias 1 -> 0
- net GND: track 254.0 -> 0.00 mm
- net Col10: track 251.4 -> 0.00 mm, vias 1 -> 0
- net LED2: track 223.9 -> 0.00 mm
- net Net-(D80-Pad2): track 218.6 -> 0.00 mm
- net Col9: track 211.1 -> 0.00 mm, vias 1 -> 0
- net LED1: track 208.3 -> 0.00 mm
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
Commit message: test
Parts:
- removed IC1: DMP1045U-7, SamacSys_Parts:SOT96P240X120-3N
- removed RF1: HolyIOT-18010-nRF52840, Keyboard Library:HolyIOT-18010-nRF52840
- removed U5: TP4056_1A_Charge, Keyboard Library:T4056 1A Charge
- added C10: C_Small, Capacitor_SMD:C_0805_2012Metric, F.Cu at (359.1, 150.4)
- added C11: 22nF, Capacitor_SMD:C_0805_2012Metric, F.Cu at (112.0, 96.5)
- added C9: 4u7, Capacitor_SMD:C_0603_1608Metric, F.Cu at (234.4, 83.1)
- added D89: 1N4148W, Diode_SMD:D_SOD-123, B.Cu at (40.2, 170.8)
- added FT1: SI2301CDS-T1-GE3, Package_TO_SOT_SMD:SOT-23, F.Cu at (130.2, 97.7)
- added H1: MountingHole_Pad, MountingHole:MountingHole_2.7mm_M2.5_DIN965_Pad, F.Cu at (334.7, 96.4)
- added J1: Conn_01x02, Connector_PinHeader_2.54mm:PinHeader_1x02_P2.54mm_Vertical, F.Cu at (101.9, 95.0)
- added J2: Conn_01x05, Connector_PinHeader_2.54mm:PinHeader_1x05_P2.54mm_Vertical, F.Cu at (378.2, 163.3)
- added L1: L, Inductor_SMD:L_0805_2012Metric, F.Cu at (361.5, 150.3)
- added R1: 5k1, Resistor_SMD:R_0805_2012Metric_Pad1.15x1.40mm_HandSolder, F.Cu at (242.9, 83.6)
- added R2: 5k1, Resistor_SMD:R_0805_2012Metric_Pad1.15x1.40mm_HandSolder, F.Cu at (237.1, 83.6)
- added R8: 10M, Resistor_SMD:R_0402_1005Metric, F.Cu at (108.6, 95.0)
- added R9: 2M2, Resistor_SMD:R_0402_1005Metric, F.Cu at (108.8, 98.5)
- added RGB_5B1: RGB, Keyboard Library:APTF1616SEEZGQBDC, F.Cu at (57.4, 172.2)
- added SW89: SW_SPST, keyswitches:Kailh_socket_MX_RGB, F.Cu at (47.8, 167.1)
- added SW90: SW_SPST, keyswitches:Kailh_socket_MX_RGB, F.Cu at (69.2, 167.1)
- added U1: TP4056_Charger, Keyboard Library:T4056 1A Charge, F.Cu at (63.9, 87.1)
- added U3: E73-2G4M08S1C-52840, nrfmicro:E73-2G4M08S1C-52840, F.Cu at (364.2, 147.3)
- C1, C15, C16, C18, C19, C2, C20, C21, C22, C3, C4, C6, C7, C8, R14, R15, R16, R17, R4, U2, U4: moved to B.Cu
- D88: value MBRS130LT3G -> NSR0340HT1G; footprint SamacSys_Parts:DIOM5436X247N -> Diode_SMD:D_SOD-323
- P1: value USB_C_Plug_USB2.0 -> USB_C_USB2.0; moved to F.Cu
- R3: value 100k -> 1M; footprint Resistor_SMD:R_0603_1608Metric -> Resistor_SMD:R_0805_2012Metric_Pad1.15x1.40mm_HandSolder
- R5: value 100k -> 3K3; footprint Resistor_SMD:R_0603_1608Metric -> Resistor_SMD:R_0402_1005Metric
- R6: value 100k -> 1k
- R7: value 100k -> 1k; footprint Resistor_SMD:R_0805_2012Metric_Pad1.15x1.40mm_HandSolder -> Resistor_SMD:R_0603_1608Metric
- moved R5 218.7 mm to (133.3, 94.3)
- moved R7 202.1 mm to (330.0, 157.7), turned to 90 degrees
- moved R3 119.1 mm to (245.8, 83.0), turned to 90 degrees
- moved RGB_7 88.4 mm to (69.2, 172.2)
- moved P1 85.7 mm to (240.2, 77.4), turned to 180 degrees
- moved C7 26.0 mm to (322.8, 154.1), turned to 90 degrees
- moved RGB_71 21.1 mm to (164.5, 226.8)
- moved C8 20.5 mm to (321.3, 154.1), turned to 90 degrees
- moved RGB_82 20.1 mm to (168.8, 226.8)
- moved RGB_48 19.9 mm to (164.5, 224.0)
- moved C6 19.9 mm to (324.4, 154.1), turned to 90 degrees
- moved RGB_42 19.9 mm to (160.2, 226.8)
- moved D23 19.1 mm to (150.3, 113.8)
- moved D25 19.0 mm to (188.5, 113.7)
- moved D24 19.0 mm to (169.5, 113.6)
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Connections:
- C1 pad 2: VCC -> PWR
- C15 pad 2: VCC -> PWR
- C16 pad 2: VCC -> V_IO
- C17 pad 1: VCC -> PWR
- C18 pad 2: VCC -> PWR
- C19 pad 2: VCC -> PWR
- C2 pad 2: VCC -> PWR
- C20 pad 2: VCC -> PWR
- C21 pad 2: VCC -> PWR
- C22 pad 2: VCC -> PWR
- C3 pad 2: VCC -> PWR
- C4 pad 2: VCC -> PWR
- C5 pad 1: VCC -> PWR
- C6 pad 2: VCC -> PWR
- C7 pad 2: VCC -> PWR
- C8 pad 2: VCC -> V_IO
- D88 pad 1: Load+ -> PWR
- D88 pad 2: Net-(D88-Pad2) -> VBUS
- P1 pad A1: Net-(P1-PadA1) -> GND
- P1 pad A12: Net-(P1-PadA1) -> GND
- P1 pad A4: Net-(P1-PadA4) -> VBUS
- P1 pad A5: (no net) -> Net-(P1-PadA5)
- P1 pad A6: (no net) -> D+
- P1 pad A7: (no net) -> D-
- P1 pad A9: Net-(P1-PadA4) -> VBUS
- P1 pad B1: Net-(P1-PadA1) -> GND
- P1 pad B12: Net-(P1-PadA1) -> GND
- P1 pad B4: Net-(P1-PadA4) -> VBUS
- P1 pad B5: (no net) -> Net-(P1-PadB5)
- P1 pad B6: (no net) -> D+
- P1 pad B7: (no net) -> D-
- P1 pad B9: Net-(P1-PadA4) -> VBUS
- P1 pad S1: Net-(P1-PadS1) -> SHIELD
- R14 pad 2: /Sheet60144165/RSET -> Net-(R14-Pad2)
- R15 pad 2: /Sheet60144165/IICRST -> IICRST
- R16 pad 2: RGB_ENABLE -> SDB
- R17 pad 2: RGB_INT -> INTB
- R3 pad 2: RGB_INT -> SHIELD
- R4 pad 2: /Sheet60144165/RSET -> Net-(R4-Pad2)
- R5 pad 1: GND -> VBUS
- R5 pad 2: /Sheet60144165/IICRST -> GND
- R6 pad 1: GND -> V_IO
- R6 pad 2: RGB_ENABLE -> I2C+
- R7 pad 1: Net-(D88-Pad2) -> I2C-
- R7 pad 2: Load- -> V_IO
- RGB_24 pad 1: CS12 -> (no net)
- RGB_24 pad 2: SW5 -> (no net)
- RGB_24 pad 3: SW4 -> (no net)
- RGB_24 pad 4: SW6 -> (no net)
- RGB_30 pad 1: CS6 -> (no net)
- RGB_30 pad 2: SW8 -> (no net)
- RGB_30 pad 3: SW7 -> (no net)
- RGB_30 pad 4: SW9 -> (no net)
- RGB_42 pad 1: CS6 -> (no net)
- RGB_42 pad 2: SW11 -> (no net)
- RGB_42 pad 3: SW10 -> (no net)
- RGB_42 pad 4: SW12 -> (no net)
- RGB_48 pad 1: CS12 -> (no net)
- RGB_48 pad 2: SW11 -> (no net)
- RGB_48 pad 3: SW10 -> (no net)
- RGB_48 pad 4: SW12 -> (no net)
- RGB_54 pad 1: CSB12 -> (no net)
- RGB_54 pad 2: SWB2 -> (no net)
- RGB_54 pad 3: SWB1 -> (no net)
- RGB_54 pad 4: SWB3 -> (no net)
- RGB_71 pad 1: CSB5 -> (no net)
- RGB_71 pad 2: SWB5 -> (no net)
- RGB_71 pad 3: SWB4 -> (no net)
- RGB_71 pad 4: SWB6 -> (no net)
- RGB_72 pad 1: CSB6 -> (no net)
- RGB_72 pad 2: SWB5 -> (no net)
- RGB_72 pad 3: SWB4 -> (no net)
- RGB_72 pad 4: SWB6 -> (no net)
- RGB_82 pad 1: CSB4 -> (no net)
- RGB_82 pad 2: SWB8 -> (no net)
- RGB_82 pad 3: SWB7 -> (no net)
- RGB_82 pad 4: SWB9 -> (no net)
- SW10 pad 1: Col9 -> Col10
- SW11 pad 1: Col10 -> Col11
- SW12 pad 1: Col11 -> Col12
- SW13 pad 1: Col12 -> Col13
- SW2 pad 1: Col1 -> Col2
- SW3 pad 1: Col2 -> Col3
- SW4 pad 1: Col3 -> Col4
- SW5 pad 1: Col4 -> Col5
- SW6 pad 1: Col5 -> Col6
- SW7 pad 1: Col6 -> Col7
- SW8 pad 1: Col7 -> Col8
- SW9 pad 1: Col8 -> Col9
- U2 pad 19: VCC -> PWR
- U2 pad 26: VCC -> PWR
- U2 pad 30: /Sheet60144165/RSET -> Net-(R4-Pad2)
- U2 pad 31: VCC -> PWR
- U2 pad 32: VCC -> V_IO
- U2 pad 33: (no net) -> RGB_SYNC
- U2 pad 36: (no net) -> PWR
- U2 pad 37: RGB_INT -> (no net)
- U2 pad 38: RGB_ENABLE -> SDB
- U2 pad 39: /Sheet60144165/IICRST -> IICRST
- U4 pad 19: VCC -> PWR
- U4 pad 26: VCC -> PWR
- U4 pad 30: /Sheet60144165/RSET -> Net-(R14-Pad2)
- U4 pad 31: VCC -> PWR
- U4 pad 32: VCC -> V_IO
- U4 pad 33: (no net) -> RGB_SYNC
- U4 pad 36: (no net) -> GND
- U4 pad 37: RGB_INT -> INTB
- U4 pad 38: RGB_ENABLE -> SDB
- U4 pad 39: /Sheet60144165/IICRST -> IICRST
Routing:
- net Col0: track 0.00 -> 434.6 mm, vias 0 -> 1
- net Row0: track 0.00 -> 426.4 mm, vias 0 -> 16
- net Row1: track 0.00 -> 425.9 mm, vias 0 -> 18
- net Row5: track 0.00 -> 412.6 mm, vias 0 -> 11
- net Row4: track 0.00 -> 406.8 mm, vias 0 -> 15
- net Col1: track 0.00 -> 404.5 mm, vias 0 -> 3
- net Col2: track 0.00 -> 393.8 mm, vias 0 -> 1
- net Row2: track 0.00 -> 386.6 mm, vias 0 -> 17
- net Col3: track 0.00 -> 346.3 mm, vias 0 -> 1
- net SWB1: track 0.00 -> 338.8 mm, vias 0 -> 9
- net SW1: track 0.00 -> 330.4 mm, vias 0 -> 10
- net Col4: track 0.00 -> 326.8 mm, vias 0 -> 1
- net SWB2: track 0.00 -> 323.0 mm, vias 0 -> 9
- net SWB3: track 0.00 -> 322.4 mm, vias 0 -> 9
- net Col5: track 0.00 -> 314.3 mm, vias 0 -> 1
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Other:
- outline, holes or cut-outs redrawn
