File: yurei.sch (KiCad schematic (older format))
At the start: 179 parts, among them SW1 SW_SPST, SW10 SW_SPST, SW11 SW_SPST, SW12 SW_SPST, SW13 SW_SPST, SW14 SW_SPST, SW15 SW_SPST, SW16 SW_SPST, SW17 SW_SPST, SW18 SW_SPST, SW19 SW_SPST, SW2 SW_SPST, SW20 SW_SPST, SW21 SW_SPST, SW22 SW_SPST, SW23 SW_SPST, SW24 SW_SPST, SW25 SW_SPST, SW26 SW_SPST, SW27 SW_SPST, SW28 SW_SPST, SW29 SW_SPST, SW3 SW_SPST, SW30 SW_SPST, SW31 SW_SPST, SW32 SW_SPST, SW33 SW_SPST, SW34 SW_SPST, SW35 SW_SPST, SW36 SW_SPST, SW37 SW_SPST, SW38 SW_SPST, SW39 SW_SPST, SW4 SW_SPST, SW40 SW_SPST, SW41 SW_SPST, SW42 SW_SPST, SW43 SW_SPST, SW44 SW_SPST, SW45 SW_SPST, SW46 SW_SPST, SW47 SW_SPST, SW48 SW_SPST, SW49 SW_SPST, SW5 SW_SPST, SW50 SW_SPST, SW51 SW_SPST, SW52 SW_SPST, SW53 SW_SPST, SW54 SW_SPST, SW55 SW_SPST, SW56 SW_SPST, SW57 SW_SPST, SW58 SW_SPST, SW59 SW_SPST, SW6 SW_SPST, SW60 SW_SPST, SW61 SW_SPST, SW62 SW_SPST, SW63 SW_SPST, SW64 SW_SPST, SW65 SW_SPST, SW66 SW_SPST, SW67 SW_SPST, SW68 SW_SPST, SW69 SW_SPST, SW7 SW_SPST, SW70 SW_SPST, SW71 SW_SPST, SW72 SW_SPST, SW73 SW_SPST, SW74 SW_SPST, SW75 SW_SPST, SW76 SW_SPST, SW77 SW_SPST, SW78 SW_SPST, SW79 SW_SPST, SW8 SW_SPST, SW80 SW_SPST, SW81 SW_SPST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

Commit message: First edit
Parts:
- added U3: Core51822B, Keyboard Library:Core51822(B), symbol Keyboard_Library:Core51822B
- D1, D10, D11, D12, D13, D14, D15, D16, D17, D18, D19, D2, D20, D21, D22, D23, D24, D25, D26, D27, D28, D29, D3, D30, D31, D32, D33, D34, D35, D36, D37, D38, D39, D4, D40, D41, D42, D43, D44, D45, D46, D47, D48, D49, D5, D50, D51, D52, D53, D54, D55, D56, D57, D58, D59, D6, D60, D61, D62, D63, D64, D65, D66, D67, D68, D69, D7, D70, D71, D72, D73, D74, D75, D76, D77, D78, D79, D8, D80, D81, D82, D83, D84, D85, D86, D87, D9: value 1N4148 -> 1N4148W; footprint yurei:D_DO-35_SOD27_P7.62mm_Horizontal -> Diode_SMD:D_SOD-123
- SW1, SW10, SW11, SW12, SW13, SW14, SW15, SW16, SW17, SW18, SW19, SW2, SW20, SW21, SW22, SW23, SW24, SW25, SW26, SW27, SW28, SW29, SW3, SW31, SW32, SW33, SW35, SW36, SW37, SW38, SW39, SW4, SW40, SW41, SW42, SW43, SW44, SW45, SW46, SW48, SW49, SW5, SW50, SW52, SW53, SW54, SW55, SW56, SW57, SW58, SW59, SW6, SW60, SW61, SW62, SW65, SW66, SW67, SW68, SW69, SW7, SW70, SW71, SW72, SW73, SW74, SW76, SW8, SW85, SW86, SW87, SW9: footprint yurei:SW_Cherry_MX_1.00u_PCB -> keyswitches:Kailh_socket_MX_RGB
- SW30: footprint yurei:SW_Cherry_MX_2.00u_PCB -> keyswitches:Kailh_socket_MX_RGB
- SW34, SW47: footprint yurei:SW_Cherry_MX_1.50u_PCB -> keyswitches:Kailh_socket_MX_RGB
- SW51: footprint yurei:SW_Cherry_MX_1.75u_PCB -> keyswitches:Kailh_socket_MX_RGB
- SW63, SW64: footprint yurei:SW_Cherry_MX_2.25u_PCB -> keyswitches:Kailh_socket_MX_RGB
- SW75: footprint yurei:SW_Cherry_MX_2.75u_PCB -> keyswitches:Kailh_socket_MX_RGB
- SW77, SW78, SW79, SW81, SW82, SW83, SW84: footprint yurei:SW_Cherry_MX_1.25u_PCB -> keyswitches:Kailh_socket_MX_RGB
- SW80: footprint yurei:SW_Cherry_MX_6.25u_PCB -> keyswitches:Kailh_socket_MX_RGB

Commit message: Added wireless circuit
nRF82840 wirelss module
TP4056 Charging/loadshare
Parts:
- removed L1, L2: LED, yurei:LED_D3.0mm, symbol yurei:LED
- removed R1, R2: 10k, yurei:R_Axial_DIN0207_L6.3mm_D2.5mm_P7.62mm_Horizontal, symbol yurei:R
- removed U1: Teensy2.0, yurei:Teensy2.0, symbol yurei:Teensy2.0_(C)
- removed U3: Core51822B, Keyboard Library:Core51822(B), symbol Keyboard_Library:Core51822B
- added D88: MBRS130LT3G, DIOM5436X247N, symbol SamacSys_Parts:MBRS130LT3G
- added IC1: DMP1045U-7, SOT96P240X120-3N, symbol SamacSys_Parts:DMP1045U-7
- added P1: USB_C_Plug_USB2.0, Keyboard Library:HRO-TYPE-C-31-M-12-Assembly, symbol Connector:USB_C_Plug_USB2.0
- added R7: 100k, Resistor_SMD:R_0805_2012Metric_Pad1.15x1.40mm_HandSolder, symbol Device:R_Small
- added RF1: HolyIOT-18010-nRF52840, Keyboard Library:HolyIOT-18010-nRF52840, symbol Keyboard_Library:HolyIOT-18010-nRF52840
- added U5: TP4056_1A_Charge, Keyboard Library:T4056 1A Charge, symbol Keyboard_Library:TP4056_1A_Charge
Connections:
- net Col0: now also RF1.12 (P0.04)
- net Col1: now also RF1.11 (P0.31)
- net Col10: now also RF1.29 (P1.01)
- net Col11: now also RF1.28 (P1.03)
- net Col12: now also RF1.21 (P0.18)
- net Col13: now also RF1.20 (P0.19)
- net Col14: now also RF1.7 (P0.02)
- net Col15: now also RF1.8 (P0.28)
- net Col16: now also RF1.9 (P0.29)
- net Col2: now also RF1.10 (P0.30)
- net Col3: now also RF1.13 (P0.05)
- net Col4: now also RF1.6 (P0.03)
- net Col5: now also RF1.36 (P0.10)
- net Col6: now also RF1.35 (P0.09)
- net Col7: now also RF1.34 (P1.06)
- net Col8: now also RF1.33 (P1.04)
- net Col9: now also RF1.30 (P1.02)
- net GND: now also RF1.1 (GND), RF1.25 (GND), RF1.37 (GND), U5.2 (GND)
- net Row0: now also RF1.27 (P1.00)
- net Row1: now also RF1.26 (P0.22)
- net Row2: now also RF1.5 (P1.15)
- net Row3: now also RF1.4 (P1.13)
- net Row4: now also RF1.3 (P1.10)
- net Row5: now also RF1.2 (P1.11)
- new net: D88.2, IC1.1 (G), R7.1, U5.1 (+5V)
- new net: IC1.3 (D), U5.6 (Load+)
- new net: P1.A1 (GND), P1.A12 (GND), P1.B1 (GND), P1.B12 (GND)
- new net: P1.A4 (VBUS), P1.A9 (VBUS), P1.B4 (VBUS), P1.B9 (VBUS)
- new net Batt+: U5.5 (Batt+)
- new net Batt-: U5.4 (Batt-)
- new net Load+: D88.1, IC1.2 (S)
- new net Load-: R7.2, U5.3 (Load-)
- no-connect marks 5 -> 23

Commit message: test
Parts:
- removed D88: MBRS130LT3G, DIOM5436X247N, symbol SamacSys_Parts:MBRS130LT3G
- removed IC1: DMP1045U-7, SOT96P240X120-3N, symbol SamacSys_Parts:DMP1045U-7
- removed P1: USB_C_Plug_USB2.0, Keyboard Library:HRO-TYPE-C-31-M-12-Assembly, symbol Connector:USB_C_Plug_USB2.0
- removed R7: 100k, Resistor_SMD:R_0805_2012Metric_Pad1.15x1.40mm_HandSolder, symbol Device:R_Small
- removed RF1: HolyIOT-18010-nRF52840, Keyboard Library:HolyIOT-18010-nRF52840, symbol Keyboard_Library:HolyIOT-18010-nRF52840
- removed U5: TP4056_1A_Charge, Keyboard Library:T4056 1A Charge, symbol Keyboard_Library:TP4056_1A_Charge
- added C10: C_Small, Capacitor_SMD:C_0805_2012Metric, symbol Device:C_Small
- added C11: 22nF, Capacitor_SMD:C_0805_2012Metric, symbol Device:C_Small
- added C9: 4u7, Capacitor_SMD:C_0603_1608Metric, symbol Device:C_Small
- added D88: NSR0340HT1G, Diode_SMD:D_SOD-323, symbol Diode:NSR0340HT1G
- added D89: 1N4148W, Diode_SMD:D_SOD-123, symbol yurei:1N4148
- added FT1: SI2301CDS-T1-GE3, Package_TO_SOT_SMD:SOT-23, symbol Device:Q_PMOS_GSD
- added H1: MountingHole_Pad, MountingHole:MountingHole_2.7mm_M2.5_DIN965_Pad, symbol Mechanical:MountingHole_Pad
- added J1: Conn_01x02, Connector_PinHeader_2.54mm:PinHeader_1x02_P2.54mm_Vertical, symbol Connector_Generic:Conn_01x02
- added J2: Conn_01x05, Connector_PinHeader_2.54mm:PinHeader_1x05_P2.54mm_Vertical, symbol Connector_Generic:Conn_01x05
- added L1: L, Inductor_SMD:L_0805_2012Metric, symbol Device:L
- added P1: USB_C_USB2.0, Keyboard Library:HRO-TYPE-C-31-M-12-Assembly, symbol Connector:USB_C_Receptacle_USB2.0
- added R1, R2: 5k1, Resistor_SMD:R_0805_2012Metric_Pad1.15x1.40mm_HandSolder, symbol Device:R
- added R3: 1M, Resistor_SMD:R_0805_2012Metric_Pad1.15x1.40mm_HandSolder, symbol Device:R
- added R5: 3K3, Resistor_SMD:R_0402_1005Metric, symbol Device:R_Small
- added R8: 10M, Resistor_SMD:R_0402_1005Metric, symbol Device:R_Small
- added R9: 2M2, Resistor_SMD:R_0402_1005Metric, symbol Device:R_Small
- added SW88: SW_Push, symbol Switch:SW_Push
- added SW89, SW90: SW_SPST, keyswitches:Kailh_socket_MX_RGB, symbol yurei:SW_SPST
- added U1: TP4056_Charger, Keyboard Library:T4056 1A Charge, symbol Keyboard_Library:TP4056_Charger
- added U3: E73-2G4M08S1C-52840, nrfmicro:E73-2G4M08S1C-52840, symbol nrfmicro:E73-2G4M08S1C-52840
Connections:
- net labels added: BATT_MON, D+, D-, I2C+, I2C-, INTB, Load, PWR, Reset, SDB, SHIELD, SWDCLK, SWDIO, VBUS, V_IO
- net labels removed: Load+, Load-, VCC
- wire segments 391 -> 467
- no-connect marks 23 -> 3
Other:
- note added: "Battery charge/protection module (100/500/1000mA)"
- note added: "Battery voltage monitor"
- note added: "Footprint needs to be confirmed!"
- note added: "If case and/or plate is conductive, connect to shield for ESD/EMC protection.\nNOTE! Full metal case is NOT recommended for wireless/BT operation!"
- note added: "J-Link connector"
- note added: "Power selector, isolates battery and charger from \nmain circuit when USB cable is inserted."
- note added: "Reset switch"
- note added: "Rprog\n10k - 130mA\n5k - 250mA\n4k - 300mA\n3k - 400mA\n2k - 580mA\n1,66 - 690mA\n1,5k - 780mA\n1,33 - 900mA\n1,2k - 1000mA"
- note added: "separate power from charger with zener? diode (no backfeed!)\nswitch??? för BT vs WL2.4Ghz"
- moved on the sheet: D1, D10, D11, D12, D13, D14, D15, D16, D17, D18, D19, D2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
